File: 005 - projetos/001 - LED resistor/primeiroProje.kicad_pcb (KiCad board)
At the start: 2 copper layers, 59 x 40 mm, 3 parts

Commit message: Feat: adjust things
Parts:
- BT1: value Battery -> 9V
- R1: value R -> 470
Changed lines of the file:
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@@
 			)
 		)
-		(property "Value" "R"
+		(property "Value" "470"
 			(at 7.62 2.37 0)
 			(layer "F.Fab")
@@
 			)
 		)
-		(property "Value" "Battery"
+		(property "Value" "9V"
 			(at 22 0 0)
 			(layer "F.Fab")
