File: 005 - projetos/001 - LED resistor/primeiroProje.kicad_sch (KiCad schematic)
At the start: 3 parts

Commit message: Feat: adjust things
Parts:
- BT1: value Battery -> 9V
- R1: value R -> 470
Changed lines of the file:
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@@
 			)
 		)
-		(property "Value" "R"
+		(property "Value" "470"
 			(at 138.4301 52.07 0)
 			(effects
@@
 			)
 		)
-		(property "Value" "Battery"
+		(property "Value" "9V"
 			(at 128.27 60.3884 0)
 			(effects
